File: QA403 Impedance Fixture.kicad_sch (KiCad schematic)
At the start: 10 parts, among them J1 NMJ6HCD2_WITH_SCREW_TERM, J2 NMJ6HCD2_WITH_SCREW_TERM, J3 Conn_Coaxial, J4 Conn_Coaxial, J5 Conn_Coaxial, J6 Conn_Coaxial

Commit message: Revision 2 fix error with jack socket connections
Rev 1 tied jack socket's tip and ring pins together.
This is OK if you use a stereo plug, but for will short
signal to ground when using a mono-plug. So a bug.
Connections:
- net A: no longer J1.R, J1.RN
- net B: no longer J2.R, J2.RN
- net COM: now also J1.R, J1.RN, J2.R, J2.RN
Changed lines of the file:
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@@
   (title_block
     (title "Speaker Impedance Fixture")
-    (date "2023-07-19")
-    (rev "1")
+    (date "2023-08-03")
+    (rev "2")
     (company "Exciton Labs Ltd")
     (comment 1 "For use with Quantasylum QA403")
@@
   (junction (at 91.44 111.76) (diameter 0) (color 0 0 0 0)
   )
+  (junction (at 91.44 116.84) (diameter 0) (color 0 0 0 0)
+  )
+  (junction (at 135.89 116.84) (diameter 0) (color 0 0 0 0)
+  )
+  (junction (at 135.89 119.38) (diameter 0) (color 0 0 0 0)
+  )
   (junction (at 128.27 124.46) (diameter 0) (color 0 0 0 0)
   )
@@
   (junction (at 171.45 76.2) (diameter 0) (color 0 0 0 0)
   )
-  (junction (at 83.82 119.38) (diameter 0) (color 0 0 0 0)
+  (junction (at 91.44 119.38) (diameter 0) (color 0 0 0 0)
   )
   (junction (at 114.3 68.58) (diameter 0) (color 0 0 0 0)
   )
-  (junction (at 83.82 116.84) (diameter 0) (color 0 0 0 0)
-  )
-  (junction (at 128.27 116.84) (diameter 0) (color 0 0 0 0)
-  )
   (junction (at 135.89 114.3) (diameter 0) (color 0 0 0 0)
   )
@@
   (junction (at 171.45 68.58) (diameter 0) (color 0 0 0 0)
   )
-  (junction (at 128.27 119.38) (diameter 0) (color 0 0 0 0)
-  )
   (junction (at 91.44 114.3) (diameter 0) (color 0 0 0 0)
   )
@@
   )
   (wire (pts (xy 181.61 60.96) (xy 181.61 68.58))
+    (stroke (width 0) (type default))
+  )
+  (wire (pts (xy 91.44 119.38) (xy 91.44 116.84))
     (stroke (width 0) (type default))
   )
@@
     (stroke (width 0) (type dash))
   )
-  (wire (pts (xy 124.46 116.84) (xy 128.27 116.84))
-    (stroke (width 0) (type default))
-  )
-  (wire (pts (xy 80.01 116.84) (xy 83.82 116.84))
+  (wire (pts (xy 135.89 116.84) (xy 135.89 114.3))
     (stroke (width 0) (type default))
   )
@@
     (stroke (width 0) (type default))
   )
-  (wire (pts (xy 83.82 121.92) (xy 83.82 119.38))
-    (stroke (width 0) (type default))
-  )
-  (wire (pts (xy 128.27 119.38) (xy 128.27 116.84))
+  (wire (pts (xy 80.01 119.38) (xy 91.44 119.38))
+    (stroke (width 0) (type default))
+  )
+  (wire (pts (xy 83.82 105.41) (xy 83.82 121.92))
+    (stroke (width 0) (type default))
+  )
+  (wire (pts (xy 124.46 119.38) (xy 135.89 119.38))
     (stroke (width 0) (type default))
   )
@@
     (stroke (width 0) (type default))
   )
+  (wire (pts (xy 80.01 116.84) (xy 91.44 116.84))
+    (stroke (width 0) (type default))
+  )
   (wire (pts (xy 190.5 66.04) (xy 190.5 72.39))
     (stroke (width 0) (type default))
@@
     (stroke (width 0) (type default))
   )
-  (wire (pts (xy 91.44 128.27) (xy 91.44 114.3))
+  (wire (pts (xy 91.44 128.27) (xy 91.44 119.38))
     (stroke (width 0) (type default))
   )
@@
     (stroke (width 0) (type default))
   )
-  (wire (pts (xy 83.82 116.84) (xy 83.82 105.41))
-    (stroke (width 0) (type default))
-  )
   (wire (pts (xy 172.72 68.58) (xy 171.45 68.58))
     (stroke (width 0) (type default))
@@
     (stroke (width 0) (type default))
   )
-  (wire (pts (xy 124.46 119.38) (xy 128.27 119.38))
-    (stroke (width 0) (type default))
-  )
   (polyline (pts (xy 213.36 119.38) (xy 234.95 119.38))
     (stroke (width 0) (type default))
@@
     (stroke (width 0) (type default))
   )
-  (wire (pts (xy 128.27 121.92) (xy 128.27 119.38))
-    (stroke (width 0) (type default))
-  )
-  (wire (pts (xy 83.82 119.38) (xy 83.82 116.84))
-    (stroke (width 0) (type default))
-  )
-  (wire (pts (xy 128.27 116.84) (xy 128.27 105.41))
+  (wire (pts (xy 128.27 105.41) (xy 128.27 121.92))
     (stroke (width 0) (type default))
   )
@@
     (stroke (width 0) (type default))
   )
+  (wire (pts (xy 135.89 119.38) (xy 135.89 116.84))
+    (stroke (width 0) (type default))
+  )
+  (wire (pts (xy 124.46 116.84) (xy 135.89 116.84))
+    (stroke (width 0) (type default))
+  )
   (wire (pts (xy 111.76 68.58) (xy 114.3 68.58))
     (stroke (width 0) (type default))
   )
+  (wire (pts (xy 91.44 116.84) (xy 91.44 114.3))
+    (stroke (width 0) (type default))
+  )
   (wire (pts (xy 171.45 68.58) (xy 171.45 76.2))
     (stroke (width 0) (type default))
   )
-  (wire (pts (xy 135.89 128.27) (xy 135.89 114.3))
+  (wire (pts (xy 135.89 128.27) (xy 135.89 119.38))
     (stroke (width 0) (type default))
   )
@@
     (stroke (width 0) (type default))
   )
-  (wire (pts (xy 80.01 119.38) (xy 83.82 119.38))
-    (stroke (width 0) (type default))
-  )
